Commit message: [update] mesh filename path

File: aizu_spider_tnk_description/urdf/CHASSIS/CHASSIS.urdf (robot description, URDF)
Before this commit: robot aizu_spider_tnk, 1 links, 0 joints
Links:
- link chassis: geometry collision mesh filename=package://aizu_spider_tnk_description/urdf/CHASSIS/-root-sh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 scale=1.0 1.0 1.0; collision mesh filename=package://aizu_spider_tnk_description/urdf/CHASSIS/-root-sh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 scale=1.0 1.0 1.0
