Commit message: [update] to use xacro

File: aizu_spider_tnk_description/urdf/CHASSIS/CHASSIS.urdf.xacro (robot description, xacro)
@@ -2,5 +2,4 @@
 <robot xmlns:xacro="http://ros.org/wiki/xacro" name="aizu_spider_tnk">
   <xacro:macro name="chassis_v0">
-    <link name="base_link"/>
     <joint name="base_link_to_chassis" type="fixed">
       <parent link="base_link"/>

Commit message: [update] inertial information

File: aizu_spider_tnk_description/urdf/CHASSIS/CHASSIS.urdf.xacro (robot description, xacro)
@@ -8,7 +8,8 @@
     <link name="chassis">
       <inertial>
-        <mass value="0.0" />
-        <origin xyz="0.0 0.0 0.0" rpy="0 -0 0" />
-        <inertia ixx="0.0" ixy="0.0" ixz="0.0" iyy="0.0" iyz="0.0" izz="0.0" />
+        <mass value="47.91109" />
+        <origin xyz="-0.08192 0 0.15046" rpy="0 -0 0" />
+        <inertia ixx="1.15503784921" ixy="0.0" ixz="-0.21517604538"
+                 iyy="2.13753698965" iyz="0.0" izz="1.94665822762" />
       </inertial>
       <visual>

Commit message: [update] chassis main belt & wheels

File: aizu_spider_tnk_description/urdf/CHASSIS/CHASSIS.urdf.xacro (robot description, xacro)
@@ -675,3 +675,27 @@
     </link>
   </xacro:macro>
+  <!-- Chassis -->
+  <xacro:chassis_v0/>
+  <!-- Main Belts -->
+  <xacro:include filename="$(find aizu_spider_tnk_description)/urdf/MAIN_BELT/MAIN_BELT.urdf.xacro"/>
+  <xacro:main_belt_v0 prefix="right">
+    <origin xyz="0 -0.14150 0.062" rpy="0 0 ${M_PI}"/>
+  </xacro:main_belt_v0>
+  <xacro:main_belt_v0 prefix="left">
+    <origin xyz="0 0.14150 0.062" rpy="0 0 0"/>
+  </xacro:main_belt_v0>
+  <!-- Wheels -->
+  <xacro:include filename="$(find aizu_spider_tnk_description)/urdf/WHEELS/WHEELS.urdf.xacro"/>
+  <xacro:track_wheel_v0 parent="chassis" prefix="FR">
+    <origin xyz="0.234 -0.146 0.062" rpy="0 0 0"/>
+  </xacro:track_wheel_v0>
+  <xacro:track_wheel_v0 parent="chassis" prefix="BR">
+    <origin xyz="-0.234 -0.146 0.062" rpy="0 0 0"/>
+  </xacro:track_wheel_v0>
+  <xacro:track_wheel_v0 parent="chassis" prefix="FL" reflect="-1">
+    <origin xyz="0.234 0.146 0.062" rpy="0 0 0"/>
+  </xacro:track_wheel_v0>
+  <xacro:track_wheel_v0 parent="chassis" prefix="BL" reflect="-1">
+    <origin xyz="-0.234 0.146 0.062" rpy="0 0 0"/>
+  </xacro:track_wheel_v0>
 </robot>
