Commit message: [update] path, link, and robot names

File: aizu_spider_tnk_description/urdf/FLIPPER/FLIPPER.urdf (robot description, URDF)
Before this commit: robot , 1 links, 0 joints
Links:
- removed link root
- added link flipper, mass 0.0; collision mesh filename=package://aizu_spider_tnk_description/urdf/FLIPPER/-root-sh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 scale=1.0 1.0 1.0; collision mesh filename=package://aizu_spider_tnk_description/urdf/FLIPPER/-root-sh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 scale=1.0 1.0 1.0
