Commit message: [update] to describe whole things

File: aizu_spider_tnk_description/urdf/FLIPPER/FLIPPER.urdf.xacro (robot description, xacro)
@@ -53,3 +53,16 @@
     </link>
   </xacro:macro>
+  <!-- Flippers -->
+  <xacro:flipper_v0 prefix="FR" reflect="-1">
+    <origin xyz="0.234 -0.22350 0.062"/>
+  </xacro:flipper_v0>
+  <xacro:flipper_v0 prefix="FL" reflect="-1">
+    <origin xyz="0.234 0.22350 0.062"/>
+  </xacro:flipper_v0>
+  <xacro:flipper_v0 prefix="BR" reflect="1">
+    <origin xyz="-0.234 -0.22350 0.062" rpy="0 0 ${M_PI}"/>
+  </xacro:flipper_v0>
+  <xacro:flipper_v0 prefix="BL" reflect="1">
+    <origin xyz="-0.234 0.22350 0.062" rpy="0 0 ${M_PI}"/>
+  </xacro:flipper_v0>
 </robot>

Commit message: [update] add subbelt & wheels

File: aizu_spider_tnk_description/urdf/FLIPPER/FLIPPER.urdf.xacro (robot description, xacro)
@@ -1,4 +1,8 @@
 <?xml version="1.0"?>
 <robot xmlns:xacro="http://ros.org/wiki/xacro" name="aizu_spider_tnk">
+  <!-- Sub Belts -->
+  <xacro:include filename="$(find aizu_spider_tnk_description)/urdf/SUB_BELT/SUB_BELT.urdf.xacro"/>
+  <!-- Wheels -->
+  <xacro:include filename="$(find aizu_spider_tnk_description)/urdf/WHEELS/WHEELS.urdf.xacro"/>
   <xacro:macro name="flipper_v0" params="prefix reflect *origin">
     <joint name="chassis_to_${prefix}_flipper" type="continuous">
@@ -52,4 +56,10 @@
       </collision>
     </link>
+    <xacro:sub_belt_v0 prefix="${prefix}"/>
+    <xacro:sub_track_wheel1_v0 parent="${prefix}_flipper" prefix="${prefix}" reflect="0">
+    </xacro:sub_track_wheel1_v0>
+    <xacro:sub_track_wheel2_v0 parent="${prefix}_flipper" prefix="${prefix}" reflect="0">
+      <origin xyz="0.29450 0 0"/>
+    </xacro:sub_track_wheel2_v0>
   </xacro:macro>
   <!-- Flippers -->

Commit message: [update] flipper subscriber

File: aizu_spider_tnk_description/urdf/FLIPPER/FLIPPER.urdf.xacro (robot description, xacro)
@@ -6,5 +6,5 @@
   <xacro:include filename="$(find aizu_spider_tnk_description)/urdf/WHEELS/WHEELS.urdf.xacro"/>
   <xacro:macro name="flipper_v0" params="prefix reflect *origin">
-    <joint name="chassis_to_${prefix}_flipper" type="continuous">
+    <joint name="${prefix}_FLIPPER" type="continuous">
       <parent link="chassis"/>
       <child link="${prefix}_flipper"/>
@@ -70,8 +70,8 @@
     <origin xyz="0.234 0.22350 0.062"/>
   </xacro:flipper_v0>
-  <xacro:flipper_v0 prefix="BR" reflect="1">
+  <xacro:flipper_v0 prefix="BR" reflect="-1">
     <origin xyz="-0.234 -0.22350 0.062" rpy="0 0 ${M_PI}"/>
   </xacro:flipper_v0>
-  <xacro:flipper_v0 prefix="BL" reflect="1">
+  <xacro:flipper_v0 prefix="BL" reflect="-1">
     <origin xyz="-0.234 0.22350 0.062" rpy="0 0 ${M_PI}"/>
   </xacro:flipper_v0>
