Commit message: [update] file path, link name, and robot name

File: aizu_spider_tnk_description/urdf/MAIN_BELT/MAIN_BELT.urdf (robot description, URDF)
Before this commit: robot , 1 links, 0 joints
Links:
- removed link root
- added link main_belt, mass 0.0; collision mesh filename=package://aizu_spider_tnk_description/urdf/MAIN_BELT/-root-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 scale=1.0 1.0 1.0; visual mesh filename=package://aizu_spider_tnk_description/urdf/MAIN_BELT/-root-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 scale=1.0 1.0 1.0
