Commit message: [update] file path, link name, and robot name

File: aizu_spider_tnk_description/urdf/MCM-4350FISH/MCM-4350FISH.urdf (robot description, URDF)
Before this commit: robot , 1 links, 0 joints
Links:
- removed link root
- added link mcm-4350fish, mass 0.0; collision mesh filename=package://aizu_spider_tnk_description/urdf/MCM-4350FISH/-ro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 scale=1.0 1.0 1.0; collision mesh filename=package://aizu_spider_tnk_description/urdf/MCM-4350FISH/-ro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 scale=1.0 1.0 1.0
