Commit message: [update] add flipper links

File: aizu_spider_tnk_description/urdf/aizu_spider_tnk.urdf.xacro (robot description, xacro)
@@ -1,6 +1,22 @@
 <?xml version="1.0"?>
 <robot xmlns:xacro="http://ros.org/wiki/xacro" name="aizu_spider_tnk">
+  <xacro:property name="M_PI" value="3.1415926535897931"/>
+  <link name="base_link"/>
+  <!-- Chassis -->
   <xacro:include filename="$(find aizu_spider_tnk_description)/urdf/CHASSIS/CHASSIS.urdf.xacro"/>
-  <link name="base_link"/>
   <xacro:chassis_v0/>
+  <!-- Flippers -->
+  <xacro:include filename="$(find aizu_spider_tnk_description)/urdf/FLIPPER/FLIPPER.urdf.xacro"/>
+  <xacro:flipper_v0 prefix="FR" reflect="-1">
+    <origin xyz="0.234 -0.22350 0.062"/>
+  </xacro:flipper_v0>
+  <xacro:flipper_v0 prefix="FL" reflect="-1">
+    <origin xyz="0.234 0.22350 0.062"/>
+  </xacro:flipper_v0>
+  <xacro:flipper_v0 prefix="BR" reflect="1">
+    <origin xyz="-0.234 -0.22350 0.062" rpy="0 0 ${M_PI}"/>
+  </xacro:flipper_v0>
+  <xacro:flipper_v0 prefix="BL" reflect="1">
+    <origin xyz="-0.234 0.22350 0.062" rpy="0 0 ${M_PI}"/>
+  </xacro:flipper_v0>
 z</robot>

Commit message: [update] to describe each macros inside of itself

File: aizu_spider_tnk_description/urdf/aizu_spider_tnk.urdf.xacro (robot description, xacro)
@@ -5,18 +5,5 @@
   <!-- Chassis -->
   <xacro:include filename="$(find aizu_spider_tnk_description)/urdf/CHASSIS/CHASSIS.urdf.xacro"/>
-  <xacro:chassis_v0/>
   <!-- Flippers -->
   <xacro:include filename="$(find aizu_spider_tnk_description)/urdf/FLIPPER/FLIPPER.urdf.xacro"/>
-  <xacro:flipper_v0 prefix="FR" reflect="-1">
-    <origin xyz="0.234 -0.22350 0.062"/>
-  </xacro:flipper_v0>
-  <xacro:flipper_v0 prefix="FL" reflect="-1">
-    <origin xyz="0.234 0.22350 0.062"/>
-  </xacro:flipper_v0>
-  <xacro:flipper_v0 prefix="BR" reflect="1">
-    <origin xyz="-0.234 -0.22350 0.062" rpy="0 0 ${M_PI}"/>
-  </xacro:flipper_v0>
-  <xacro:flipper_v0 prefix="BL" reflect="1">
-    <origin xyz="-0.234 0.22350 0.062" rpy="0 0 ${M_PI}"/>
-  </xacro:flipper_v0>
-z</robot>
+</robot>

Commit message: [add] to use common xacro file

File: aizu_spider_tnk_description/urdf/aizu_spider_tnk.urdf.xacro (robot description, xacro)
@@ -1,5 +1,5 @@
 <?xml version="1.0"?>
 <robot xmlns:xacro="http://ros.org/wiki/xacro" name="aizu_spider_tnk">
-  <xacro:property name="M_PI" value="3.1415926535897931"/>
+  <xacro:include filename="$(find aizu_spider_tnk_description)/urdf/common.xacro"/>
   <link name="base_link"/>
   <!-- Chassis -->

Commit message: [update] to load basical model

File: aizu_spider_tnk_description/urdf/aizu_spider_tnk.urdf.xacro (robot description, xacro)
@@ -1,9 +1,5 @@
 <?xml version="1.0"?>
 <robot xmlns:xacro="http://ros.org/wiki/xacro" name="aizu_spider_tnk">
-  <xacro:include filename="$(find aizu_spider_tnk_description)/urdf/common.xacro"/>
-  <link name="base_link"/>
-  <!-- Chassis -->
-  <xacro:include filename="$(find aizu_spider_tnk_description)/urdf/CHASSIS/CHASSIS.urdf.xacro"/>
-  <!-- Flippers -->
-  <xacro:include filename="$(find aizu_spider_tnk_description)/urdf/FLIPPER/FLIPPER.urdf.xacro"/>
+  <!-- Load Basic -->
+  <include filename="$(find aizu_spider_tnk_description)/urdf/aizu_spider_basic.urdf.xacro"/>
 </robot>
