Commit message: [add] common color

File: aizu_spider_tnk_description/urdf/common.xacro (robot description, xacro)
@@ -4,4 +4,7 @@
     <color rgba="1 1 0.752941 1"/>
   </material>
+  <material name="orange">
+    <color rgba="0.73 0.36 0.02 1"/>
+  </material>
   <xacro:property name="M_PI" value="3.1415926535897931"/>
 </robot>
