Commit message: [add] jaco2 xacro

File: aizu_spider_tnk_description/urdf/aizu_spider.urdf.xacro (robot description, xacro)
@@ -5,3 +5,12 @@
   <!-- Load Sensors -->
   <xacro:include filename="$(find aizu_spider_tnk_description)/urdf/sensors/sensors.urdf.xacro"/>
+  <xacro:include filename="$(find kinova_description)/urdf/j2n6s300_standalone.xacro"/>
+  <joint name="chassis_to_jaco_link" type="fixed">
+    <parent link="chassis"/>
+    <child link="jaco_link"/>
+    <origin xyz=" -0.06320 -0.094 0.5150" rpy="${M_PI/2} ${M_PI/2} ${M_PI/2}"/>
+    <!-- <origin xyz=" -0.06320 -0.094 0.5150" rpy="0 0 0"/> -->
+  </joint>
+  <link name="jaco_link"/>
+  <xacro:j2n6s300  base_parent="jaco_link"/>
 </robot>

Commit message: [update] jaco_link rotation

File: aizu_spider_tnk_description/urdf/aizu_spider.urdf.xacro (robot description, xacro)
@@ -9,5 +9,5 @@
     <parent link="chassis"/>
     <child link="jaco_link"/>
-    <origin xyz=" -0.06320 -0.094 0.5150" rpy="${M_PI/2} ${M_PI/2} ${M_PI/2}"/>
+    <origin xyz=" -0.06320 -0.094 0.5150" rpy="${M_PI/2} 0 ${M_PI/2}"/>
     <!-- <origin xyz=" -0.06320 -0.094 0.5150" rpy="0 0 0"/> -->
   </joint>

Commit message: [add] kinect link

File: aizu_spider_tnk_description/urdf/aizu_spider.urdf.xacro (robot description, xacro)
@@ -10,8 +10,16 @@
     <parent link="chassis"/>
     <child link="jaco_link"/>
-    <origin xyz=" -0.06320 -0.094 0.5150" rpy="${M_PI/2} 0 ${M_PI/2}"/>
+    <origin xyz="-0.06320 -0.094 0.5150" rpy="${M_PI/2} 0 ${M_PI/2}"/>
     <!-- <origin xyz=" -0.06320 -0.094 0.5150" rpy="0 0 0"/> -->
   </joint>
   <link name="jaco_link"/>
   <xacro:j2n6s300  base_parent="jaco_link"/>
+  <!-- God of  Kinect -->
+  <joint name="_to_ARM_Kinect" type="fixed">
+    <parent link="j2n6s300_end_effector"/>
+    <child link="ARM_Kinect"/>
+    <!-- <origin xyz="0.03116 0 0.11498" rpy="0 0 0"/> -->
+    <origin xyz="0 0 0" rpy="0 0 ${M_PI/2}"/>
+  </joint>
+  <link name="ARM_Kinect"/>
 </robot>

Commit message: [update] to add kinect urdf on sensor xacro file

File: aizu_spider_tnk_description/urdf/aizu_spider.urdf.xacro (robot description, xacro)
@@ -15,11 +15,3 @@
   <link name="jaco_link"/>
   <xacro:j2n6s300  base_parent="jaco_link"/>
-  <!-- God of  Kinect -->
-  <joint name="_to_ARM_Kinect" type="fixed">
-    <parent link="j2n6s300_end_effector"/>
-    <child link="ARM_Kinect"/>
-    <!-- <origin xyz="0.03116 0 0.11498" rpy="0 0 0"/> -->
-    <origin xyz="0 0 0" rpy="0 0 ${M_PI/2}"/>
-  </joint>
-  <link name="ARM_Kinect"/>
 </robot>

File: aizu_spider_tnk_description/urdf/sensors/sensors.urdf.xacro (robot description, xacro)
@@ -26,3 +26,11 @@
   <xacro:include filename="$(find aizu_spider_tnk_description)/urdf/sensors/ACC_SENSOR/ACC_SENSOR.urdf.xacro"/>
   <xacro:acc_sensor_v0/>
+  <!-- God of  Kinect -->
+  <joint name="_to_ARM_Kinect" type="fixed">
+    <parent link="j2n6s300_end_effector"/>
+    <child link="ARM_Kinect"/>
+    <!-- <origin xyz="0.03116 0 0.11498" rpy="0 0 0"/> -->
+    <origin xyz="0 0 0" rpy="0 0 ${M_PI/2}"/>
+  </joint>
+  <link name="ARM_Kinect"/>
 </robot>
