Commit message: [update] file path

File: aizu_spider_tnk_description/urdf/sensors/UTM-30LN/UTM-30LN.urdf.xacro (robot description, xacro)
@@ -16,5 +16,5 @@
         <origin xyz="0.0 0.0 0.0" rpy="0.0 -0.0 0.0" />
         <geometry>
-          <mesh filename="package://aizu_spider_tnk_description/urdf/UTM-30LN/-root-shape-0.dae" scale="1.0 1.0 1.0" />
+          <mesh filename="package://aizu_spider_tnk_description/urdf/sensors/UTM-30LN/-root-shape-0.dae" scale="1.0 1.0 1.0" />
         </geometry>
       </visual>
@@ -22,5 +22,5 @@
         <origin xyz="0.0 0.0 0.0" rpy="0.0 -0.0 0.0" />
         <geometry>
-          <mesh filename="package://aizu_spider_tnk_description/urdf/UTM-30LN/-root-shape-0.dae" scale="1.0 1.0 1.0" />
+          <mesh filename="package://aizu_spider_tnk_description/urdf/sensors/UTM-30LN/-root-shape-0.dae" scale="1.0 1.0 1.0" />
         </geometry>
       </collision>
