Commit message: [update] link name

File: aizu_spider_tnk_description/urdf/sensors/MCM-4350FISH/MCM-4350FISH.urdf.xacro (robot description, xacro)
@@ -2,10 +2,10 @@
 <robot xmlns:xacro="http://ros.org/wiki/xacro" name="aizu_spider">
   <xacro:macro name="mcm-4350fish_v0" params="prefix *origin">
-    <joint name="chassis_to_${prefix}_mcm-4350fish" type="fixed">
+    <joint name="chassis_to_${prefix}_CAMERA" type="fixed">
       <parent link="chassis"/>
-      <child link="${prefix}_mcm-4350fish"/>
+      <child link="${prefix}_CAMERA"/>
       <insert_block name="origin"/>
     </joint>
-    <link name="${prefix}_mcm-4350fish">
+    <link name="${prefix}_CAMERA">
       <inertial>
         <mass value="0.0" />

File: aizu_spider_tnk_description/urdf/sensors/UTM-30LN/UTM-30LN.urdf.xacro (robot description, xacro)
@@ -2,10 +2,16 @@
 <robot xmlns:xacro="http://ros.org/wiki/xacro" name="aizu_spider">
   <xacro:macro name="utm-30ln_v0" params="prefix *origin">
-    <joint name="chassis_to_${prefix}_utm-30ln" type="fixed">
+    <joint name="virtual_${prefix}_LRF_to_${prefix}_LRF" type="fixed">
+      <parent link="virtual_${prefix}_LRF"/>
+      <child link="${prefix}_LRF"/>
+      <origin rpy="${-M_PI/2} ${M_PI/2} 0"/>
+    </joint>
+    <link name="${prefix}_LRF"/>
+    <joint name="chassis_to_virtual_${prefix}_LRF" type="fixed">
       <parent link="chassis"/>
-      <child link="${prefix}_utm-30ln"/>
+      <child link="virtual_${prefix}_LRF"/>
       <insert_block name="origin"/>
     </joint>
-    <link name="${prefix}_utm-30ln">
+    <link name="virtual_${prefix}_LRF">
       <inertial>
         <mass value="0.0" />

File: aizu_spider_tnk_description/urdf/sensors/sensors.urdf.xacro (robot description, xacro)
@@ -3,20 +3,24 @@
   <!-- Camera -->
   <xacro:include filename="$(find aizu_spider_tnk_description)/urdf/sensors/MCM-4350FISH/MCM-4350FISH.urdf.xacro"/>
-  <xacro:mcm-4350fish_v0 prefix="front">
+  <xacro:mcm-4350fish_v0 prefix="FRONT">
     <origin xyz="0.25470 0 0.13550" rpy="${M_PI/2} 0 ${-M_PI/2}"/>
   </xacro:mcm-4350fish_v0>
-  <xacro:mcm-4350fish_v0 prefix="left">
+  <xacro:mcm-4350fish_v0 prefix="LEFT">
     <origin xyz="0 0.17850 0.04450" rpy="${M_PI/2} 0 0"/>
   </xacro:mcm-4350fish_v0>
-  <xacro:mcm-4350fish_v0 prefix="right">
+  <xacro:mcm-4350fish_v0 prefix="RIGHT">
     <origin xyz="0 -0.17850 0.04450" rpy="${M_PI/2} 0 ${M_PI}"/>
   </xacro:mcm-4350fish_v0>
-  <xacro:mcm-4350fish_v0 prefix="back">
+  <xacro:mcm-4350fish_v0 prefix="BACK">
     <origin xyz="-0.35670 0 0.094" rpy="${M_PI/2} 0 ${M_PI/2}"/>
   </xacro:mcm-4350fish_v0>
   <!-- LRF -->
   <xacro:include filename="$(find aizu_spider_tnk_description)/urdf/sensors/UTM-30LN/UTM-30LN.urdf.xacro"/>
-  <xacro:utm-30ln_v0 prefix="front">
+  <xacro:utm-30ln_v0 prefix="FRONT">
     <origin xyz="0.23415 0 0.19750" rpy="${M_PI/2} 0 ${-M_PI/2}"/>
   </xacro:utm-30ln_v0>
+  <xacro:include filename="$(find aizu_spider_tnk_description)/urdf/sensors/LIDAR-VLP16/LIDAR-VLP16.urdf.xacro"/>
+  <xacro:lidar-vlp16_v0 prefix="TOP">
+    <origin xyz="0 0 0.7" rpy="${M_PI/2} 0 ${-M_PI/2}"/>
+  </xacro:lidar-vlp16_v0>
 </robot>
