Commit message: [update] joint name to satisfy cnoid JACO2

File: kinova_description/urdf/kinova_common.xacro (robot description, xacro)
@@ -91,5 +91,5 @@
     <xacro:macro name="kinova_finger" params="prefix finger_number hand finger_origin_xyz finger_origin_rpy">
         <xacro:kinova_armlink link_name="${prefix}link_finger_${finger_number}" link_mesh="finger_proximal" mesh_no="57"/>
-        <joint name="${prefix}joint_finger_${finger_number}" type="revolute">
+        <joint name="FINGER${finger_number}" type="revolute">
             <parent link="${hand}"/>
             <child link="${prefix}link_finger_${finger_number}"/>
