Commit message: [update] to load whole cameras

File: aizu_spider_tnk_description/urdf/sensors/sensors.urdf.xacro (robot description, xacro)
@@ -1,3 +1,16 @@
 <?xml version="1.0"?>
 <robot xmlns:xacro="http://ros.org/wiki/xacro" name="aizu_spider">
-</robot>>
+  <xacro:include filename="$(find aizu_spider_tnk_description)/urdf/sensors/MCM-4350FISH/MCM-4350FISH.urdf.xacro"/>
+  <xacro:mcm-4350fish_v0 prefix="front">
+    <origin xyz="0.25470 0 0.13550" rpy="${M_PI/2} 0 ${-M_PI/2}"/>
+  </xacro:mcm-4350fish_v0>
+  <xacro:mcm-4350fish_v0 prefix="left">
+    <origin xyz="0 0.17850 0.04450" rpy="${M_PI/2} 0 0"/>
+  </xacro:mcm-4350fish_v0>
+  <xacro:mcm-4350fish_v0 prefix="right">
+    <origin xyz="0 -0.17850 0.04450" rpy="${M_PI/2} 0 ${M_PI}"/>
+  </xacro:mcm-4350fish_v0>
+  <xacro:mcm-4350fish_v0 prefix="back">
+    <origin xyz="-0.35670 0 0.094" rpy="${M_PI/2} 0 ${M_PI/2}"/>
+  </xacro:mcm-4350fish_v0>
+</robot>

Commit message: [update] to load LRF

File: aizu_spider_tnk_description/urdf/sensors/sensors.urdf.xacro (robot description, xacro)
@@ -1,4 +1,5 @@
 <?xml version="1.0"?>
 <robot xmlns:xacro="http://ros.org/wiki/xacro" name="aizu_spider">
+  <!-- Camera -->
   <xacro:include filename="$(find aizu_spider_tnk_description)/urdf/sensors/MCM-4350FISH/MCM-4350FISH.urdf.xacro"/>
   <xacro:mcm-4350fish_v0 prefix="front">
@@ -14,3 +15,8 @@
     <origin xyz="-0.35670 0 0.094" rpy="${M_PI/2} 0 ${M_PI/2}"/>
   </xacro:mcm-4350fish_v0>
+  <!-- LRF -->
+  <xacro:include filename="$(find aizu_spider_tnk_description)/urdf/sensors/UTM-30LN/UTM-30LN.urdf.xacro"/>
+  <xacro:utm-30ln_v0 prefix="front">
+    <origin xyz="0.23415 0 0.19750" rpy="${M_PI/2} 0 ${-M_PI/2}"/>
+  </xacro:utm-30ln_v0>
 </robot>

Commit message: [update]

File: aizu_spider_tnk_description/urdf/sensors/sensors.urdf.xacro (robot description, xacro)
@@ -27,5 +27,5 @@
   <xacro:acc_sensor_v0/>
   <!-- God of  Kinect -->
-  <joint name="_to_ARM_Kinect" type="fixed">
+  <joint name="j2n6s300_end_effector_to_ARM_Kinect" type="fixed">
     <parent link="j2n6s300_end_effector"/>
     <child link="ARM_Kinect"/>
