Commit message: Update TOHOKU ARM

File: double_arm_tnk_description/urdf/TOHOKU_ARM.urdf.xacro (robot description, xacro)
@@ -1,6 +1,41 @@
 <?xml version="1.0"?>
 <robot  xmlns:xacro="http://ros.org/wiki/xacro">
+  <!-- == Material == -->
+  <material name="mframe_color">
+    <color rgba="0.2 0.2 0.2 1"/>
+  </material>
+  <material name="block_color">
+    <color rgba="1 0.85 0.33 1"/>
+  </material>
+  <material name="boom_color">
+    <color rgba="1 0.85 0.33 1"/>
+  </material>
+  <material name="arm_color">
+    <color rgba="1 0.85 0.33 1"/>
+  </material>
+  <material name="tohku_pitch_color">
+    <color rgba="0.5 0.5 0.5 1"/>
+  </material>
+  <material name="tohku_roll_color">
+    <color rgba="0.39 0.51 0.91 1"/>
+  </material>
+  <material name="tohku_tip_color">
+    <color rgba="0.7 0.7 0.7 1"/>
+  </material>
   <!-- Link -->
   <link name="MFRAME">
+    <visual>
+      <origin rpy="${M_PI/2} 0 ${M_PI}"/>
+      <material name="mframe_color"/>
+      <geometry>
+        <mesh filename="package://double_arm_tnk_description/meshes/middleframe.stl"/>
+      </geometry>
+    </visual>
+    <collision>
+      <origin rpy="${M_PI/2} 0 ${M_PI}"/>
+      <geometry>
+        <mesh filename="package://double_arm_tnk_description/meshes/middleframe.stl"/>
+      </geometry>
+    </collision>
     <inertial>
       <mass value="1e-06" />
@@ -10,4 +45,17 @@
   </link>
   <link name="BLOCK">
+    <visual>
+      <origin rpy="${M_PI/2} 0 ${M_PI}"/>
+      <material name="block_color"/>
+      <geometry>
+        <mesh filename="package://double_arm_tnk_description/meshes/swingbrkt.stl"/>
+      </geometry>
+    </visual>
+    <collision>
+      <origin rpy="${M_PI/2} 0 ${M_PI}"/>
+      <geometry>
+        <mesh filename="package://double_arm_tnk_description/meshes/swingbrkt.stl"/>
+      </geometry>
+    </collision>
     <inertial>
       <mass value="1e-06" />
@@ -17,4 +65,15 @@
   </link>
   <link name="BOOM">
+    <visual>
+      <material name="boom_color"/>
+      <geometry>
+        <mesh filename="package://double_arm_tnk_description/meshes/cp_boom.stl"/>
+      </geometry>
+    </visual>
+    <collision>
+      <geometry>
+        <mesh filename="package://double_arm_tnk_description/meshes/cp_boom.stl"/>
+      </geometry>
+    </collision>
     <inertial>
       <mass value="88.2695650987" />
@@ -22,72 +81,17 @@
       <inertia ixx="1.48138597730672" ixy="0.1902362002908" ixz="1.05546586084014e-15" iyy="31.4435403431583" iyz="-2.05305944696362e-17" izz="32.5752155940256" />
     </inertial>
-    <collision>
-      <origin xyz="0.0 0.0 0.0" rpy="1.57079632679 0.375245789179 -3.14159265359" />
-      <geometry>
-        <cylinder radius="0.05" length="0.116" />
-      </geometry>
-    </collision>
-    <collision>
-      <origin xyz="0.4186879055919116 -1.9907224074340133e-16 0.16492555202593392" rpy="1.13579022766e-16 -0.375245789179 3.14159265359" />
-      <geometry>
-        <box size="0.9 0.116 0.1" />
-      </geometry>
-    </collision>
-    <collision>
-      <origin xyz="0.40419402094470985 -2.1228539612808136e-16 0.1948991622161264" rpy="3.02966782347e-17 -0.449422282389 3.14159265359" />
-      <geometry>
-        <box size="0.895 0.116 0.1" />
-      </geometry>
-    </collision>
-    <collision>
-      <origin xyz="1.1879713766505169 -4.354270489073068e-16 0.18116085136942053" rpy="8.75683157457e-17 -0.296705972839 3.14159265359" />
-      <geometry>
-        <box size="0.899 0.116 0.09" />
-      </geometry>
-    </collision>
-    <collision>
-      <origin xyz="1.1953232786166952 -4.750760030961959e-16 0.22230935726550022" rpy="1.15686232084e-16 -0.381354441561 3.14159265359" />
-      <geometry>
-        <box size="0.92 0.116 0.09" />
-      </geometry>
-    </collision>
-    <collision>
-      <origin xyz="1.7600000000000025 -0.05325000000000048 2.3733810657253497e-16" rpy="1.57079632679 -0.296705972839 3.14159265359" />
-      <geometry>
-        <cylinder radius="0.04" length="0.0095" />
-      </geometry>
-    </collision>
-    <collision>
-      <origin xyz="1.6834956195229596 -0.05325000000000048 0.023389736377819183" rpy="8.75683157457e-17 -0.296705972839 3.14159265359" />
-      <geometry>
-        <box size="0.16 0.0095 0.08" />
-      </geometry>
-    </collision>
-    <collision>
-      <origin xyz="1.68568840730838 -0.053250000000000484 0.030562022047541958" rpy="1.16593465255e-16 -0.383972435439 3.14159265359" />
-      <geometry>
-        <box size="0.16 0.0095 0.08" />
-      </geometry>
-    </collision>
-    <collision>
-      <origin xyz="1.7600000000000025 0.05324999999999962 1.9373756672733388e-16" rpy="1.57079632679 -0.296705972839 3.14159265359" />
-      <geometry>
-        <cylinder radius="0.04" length="0.0095" />
-      </geometry>
-    </collision>
-    <collision>
-      <origin xyz="1.6834956195229596 0.05324999999999962 0.023389736377819142" rpy="8.75683157457e-17 -0.296705972839 3.14159265359" />
-      <geometry>
-        <box size="0.16 0.0095 0.08" />
-      </geometry>
-    </collision>
-    <collision>
-      <origin xyz="1.68568840730838 0.05324999999999961 0.030562022047541916" rpy="1.16593465255e-16 -0.383972435439 3.14159265359" />
-      <geometry>
-        <box size="0.16 0.0095 0.08" />
-      </geometry>
-    </collision>
   </link>
   <link name="ARM">
+    <visual>
+      <material name="arm_color"/>
+      <geometry>
+        <mesh filename="package://double_arm_tnk_description/meshes/cp_arm.stl"/>
+      </geometry>
+    </visual>
+    <collision>
+      <geometry>
+        <mesh filename="package://double_arm_tnk_description/meshes/cp_arm.stl"/>
+      </geometry>
+    </collision>
     <inertial>
       <mass value="53.7797060658" />
@@ -95,66 +99,19 @@
       <inertia ixx="0.35420506763418" ixy="-0.59676584437886" ixz="1.78134245842626e-16" iyy="5.16579159038522" iyz="6.97110293472855e-17" izz="5.39850890239257" />
     </inertial>
-    <collision>
-      <origin xyz="-0.24300000000000033 -1.5533242026099217e-17 0.08450000000000005" rpy="1.57079632679 -0.336848545635 3.14159265359" />
-      <geometry>
-        <cylinder radius="0.0296" length="0.083" />
-      </geometry>
-    </collision>
-    <collision>
-      <origin xyz="-0.11936207534259712 -7.359996381010075e-18 0.04120261455456779" rpy="2.17510348387e-17 -0.336848545635 3.14159265359" />
-      <geometry>
-        <box size="0.262 0.083 0.0592" />
-      </geometry>
-    </collision>
-    <collision>
-      <origin xyz="-0.09103700321555463 -6.195145466645663e-17 0.09485604211514259" rpy="2.17510348387e-17 -0.336848545635 3.14159265359" />
-      <geometry>
-        <box size="0.14 0.083 0.07" />
-      </geometry>
-    </collision>
-    <collision>
-      <origin xyz="-0.09112686398426773 -1.2057425648815144e-16 0.16088422976470257" rpy="1.46430338297e-16 -0.466002910282 3.14159265359" />
-      <geometry>
-        <box size="0.34 0.083 0.0592" />
-      </geometry>
-    </collision>
-    <collision>
-      <origin xyz="0.05700000000000005 -2.233934448755695e-16 0.23580000000000023" rpy="1.57079632679 -1.02101761242 3.14159265359" />
-      <geometry>
-        <cylinder radius="0.0296" length="0.083" />
-      </geometry>
-    </collision>
-    <collision>
-      <origin xyz="0.03581365767610803 -1.1292183821525238e-16 0.11726250003085589" rpy="1.14524417827e-16 -1.02101761242 3.14159265359" />
-      <geometry>
-        <box size="0.18 0.083 0.2192" />
-      </geometry>
-    </collision>
-    <collision>
-      <origin xyz="0.47950000000000065 -1.174436280382313e-16 5.898059818321144e-17" rpy="0.0 -0.0 3.14159265359" />
-      <geometry>
-        <box size="0.971 0.083 0.06" />
-      </geometry>
-    </collision>
-    <collision>
-      <origin xyz="0.12400000000000017 -6.589837740685943e-17 0.04000000000000006" rpy="0.0 -0.0 3.14159265359" />
-      <geometry>
-        <box size="0.4 0.083 0.06" />
-      </geometry>
-    </collision>
-    <collision>
-      <origin xyz="0.9650000000000013 -2.363568322354394e-16 1.1817841611771973e-16" rpy="1.57079632679 -0.0872664625993 3.14159265359" />
-      <geometry>
-        <cylinder radius="0.03" length="0.083" />
-      </geometry>
-    </collision>
-    <collision>
-      <origin xyz="0.4813474740764582 -1.5547861078879205e-16 0.04231411310398813" rpy="-1.40826537065e-17 -0.0872664625997 -3.14159265359" />
-      <geometry>
-        <box size="0.971 0.083 0.06" />
-      </geometry>
-    </collision>
   </link>
   <link name="TOHKU_PITCH">
+    <visual>
+      <origin rpy="${-M_PI/2} ${-M_PI/2} 0"/>
+      <material name="tohku_pitch_color"/>
+      <geometry>
+        <mesh filename="package://double_arm_tnk_description/meshes/tohku_hand_pitch.stl"/>
+      </geometry>
+    </visual>
+    <collision>
+      <origin rpy="${-M_PI/2} ${-M_PI/2} 0"/>
+      <geometry>
+        <mesh filename="package://double_arm_tnk_description/meshes/tohku_hand_pitch.stl"/>
+      </geometry>
+    </collision>
     <inertial>
       <mass value="1e-06" />
@@ -164,4 +121,17 @@
   </link>
   <link name="TOHKU_ROLL">
+    <visual>
+      <origin rpy="${-M_PI/2} ${-M_PI/2} 0"/>
+      <material name="tohku_roll_color"/>
+      <geometry>
+        <mesh filename="package://double_arm_tnk_description/meshes/tohku_hand_roll.stl"/>
+      </geometry>
+    </visual>
+    <collision>
+      <origin rpy="${-M_PI/2} ${-M_PI/2} 0"/>
+      <geometry>
+        <mesh filename="package://double_arm_tnk_description/meshes/tohku_hand_roll.stl"/>
+      </geometry>
+    </collision>
     <inertial>
       <mass value="1e-06" />
@@ -171,4 +141,17 @@
   </link>
   <link name="TOHKU_TIP_01">
+    <visual>
+      <origin rpy="${-M_PI/2} ${-M_PI/2} 0"/>
+      <material name="tohku_tip_color"/>
+      <geometry>
+        <mesh filename="package://double_arm_tnk_description/meshes/tohku_hand_tip.stl"/>
+      </geometry>
+    </visual>
+    <collision>
+      <origin rpy="${-M_PI/2} ${-M_PI/2} 0"/>
+      <geometry>
+        <mesh filename="package://double_arm_tnk_description/meshes/tohku_hand_tip.stl"/>
+      </geometry>
+    </collision>
     <inertial>
       <mass value="1e-06" />
@@ -178,4 +161,17 @@
   </link>
   <link name="TOHKU_TIP_02">
+    <visual>
+      <origin rpy="${-M_PI/2} ${-M_PI/2} 0"/>
+      <material name="tohku_tip_color"/>
+      <geometry>
+        <mesh filename="package://double_arm_tnk_description/meshes/tohku_hand_tip.stl"/>
+      </geometry>
+    </visual>
+    <collision>
+      <origin rpy="${-M_PI/2} ${-M_PI/2} 0"/>
+      <geometry>
+        <mesh filename="package://double_arm_tnk_description/meshes/tohku_hand_tip.stl"/>
+      </geometry>
+    </collision>
     <inertial>
       <mass value="1e-06" />
