Commit message: Update MANI ARM

File: double_arm_tnk_description/urdf/MANI_ARM.urdf.xacro (robot description, xacro)
@@ -1,6 +1,59 @@
 <?xml version="1.0"?>
 <robot xmlns:xacro="http://ros.org/wiki/xacro">
+  <!-- Material -->
+  <material name="uframe_color">
+    <color rgba="1 0.85 0.33 1"/>
+  </material>
+  <material name="mnp_swing_color">
+    <color rgba="1 0.85 0.33 1"/>
+  </material>
+  <material name="maniboom_color">
+    <color rgba="1 0.85 0.33 1"/>
+  </material>
+  <material name="maniarm_color">
+    <color rgba="1 0.85 0.33 1"/>
+  </material>
+  <material name="manielbow_color">
+    <color rgba="0.89 0.89 1 1"/>
+  </material>
+  <material name="yawjoint_color">
+    <color rgba="0.54 0.46 0.62 1"/>
+  </material>
+  <material name="handbase_color">
+    <color rgba="0.4 0.4 0.4 0.9"/>
+  </material>
+  <material name="pushrod_color">
+    <color rgba="0.87 0.87 0.91 1"/>
+  </material>
+  <material name="handslnk_i_color">
+    <color rgba="0.4 0.4 0.4 1"/>
+  </material>
+  <material name="handslnk_o_color">
+    <color rgba="0.4 0.4 0.4 1"/>
+  </material>
+  <material name="manifng_color">
+    <color rgba="0.2 0.2 0.2 1"/>
+  </material>
+  <material name="handtip_color">
+    <color rgba="0.9 0.9 0.9 1"/>
+  </material>
+  <material name="handlnk_color">
+    <color rgba="0.87 0.7426 0.79 1"/>
+  </material>
   <!-- Link -->
   <link name="UFRAME">
+    <visual>
+      <origin rpy="${M_PI/2} 0 0"/>
+      <material name="uframe_color"/>
+      <geometry>
+        <mesh filename="package://double_arm_tnk_description/meshes/frame_marge.stl"/>
+      </geometry>
+    </visual>
+    <collision>
+      <origin rpy="${M_PI/2} 0 0"/>
+      <geometry>
+        <mesh filename="package://double_arm_tnk_description/meshes/frame_marge.stl"/>
+      </geometry>
+    </collision>
     <inertial>
       <mass value="1e-06" />
@@ -10,4 +63,17 @@
   </link>
   <link name="MNP_SWING">
+    <visual>
+      <origin rpy="${M_PI/2} 0 ${M_PI}"/>
+      <material name="mnp_swing_color"/>
+      <geometry>
+        <mesh filename="package://double_arm_tnk_description/meshes/mani_swgbrkt_v7.stl"/>
+      </geometry>
+    </visual>
+    <collision>
+      <origin rpy="${M_PI/2} 0 ${M_PI}"/>
+      <geometry>
+        <mesh filename="package://double_arm_tnk_description/meshes/mani_swgbrkt_v7.stl"/>
+      </geometry>
+    </collision>
     <inertial>
       <mass value="1e-06" />
@@ -17,4 +83,15 @@
   </link>
   <link name="MANIBOOM">
+    <visual>
+      <material name="maniboom_color"/>
+      <geometry>
+        <mesh filename="package://double_arm_tnk_description/meshes/mani_boom_v7_2.stl"/>
+      </geometry>
+    </visual>
+    <collision>
+      <geometry>
+        <mesh filename="package://double_arm_tnk_description/meshes/mani_boom_v7_2.stl"/>
+      </geometry>
+    </collision>
     <inertial>
       <mass value="36.291074" />
@@ -22,168 +99,17 @@
       <inertia ixx="0.11028539" ixy="0.04398908" ixz="0.0" iyy="7.0046174" iyz="0.0" izz="6.9737013" />
     </inertial>
-    <collision>
-      <origin xyz="0.0 0.0 0.0" rpy="3.14159265359 1.22464679915e-16 3.14159265359" />
-      <geometry>
-        <cylinder radius="0.035" length="0.18" />
-      </geometry>
-    </collision>
-    <collision>
-      <origin xyz="0.09360186960740366 0.41357191636521845 -3.813787642366294e-16" rpy="1.57079632679 -9.74498259865e-14 2.93128047872" />
-      <geometry>
-        <box size="0.07 0.115 0.849" />
-      </geometry>
-    </collision>
-    <collision>
-      <origin xyz="0.13449564031850803 1.0875085889329599 -9.917384094630197e-16" rpy="1.57079632679 1.72251102271e-13 -2.98887634404" />
-      <geometry>
-        <box size="0.08 0.115 0.55" />
-      </geometry>
-    </collision>
-    <collision>
-      <origin xyz="0.017373789739834413 0.22015174637071627 -1.997831702439419e-16" rpy="1.57079632679 -1.69711467102e-13 2.97578637465" />
-      <geometry>
-        <box size="0.03 0.115 0.4" />
-      </geometry>
-    </collision>
-    <collision>
-      <origin xyz="0.07702917045091942 0.5975639454389267 -5.452515119623752e-16" rpy="1.57079632679 -1.69681976803e-12 3.08923277603" />
-      <geometry>
-        <box size="0.08 0.115 0.5" />
-      </geometry>
-    </collision>
-    <collision>
-      <origin xyz="0.0860000000000008 1.0775000000000017 -9.779052824825384e-16" rpy="1.57079632679 1.34266957257e-15 3.14159265359" />
-      <geometry>
-        <box size="0.08 0.115 0.575" />
-      </geometry>
-    </collision>
-    <collision>
-      <origin xyz="0.13600000000000073 0.7900000000000013 -7.242432995517537e-16" rpy="1.57079632679 1.34266957257e-15 3.14159265359" />
-      <geometry>
-        <box size="0.05 0.115 0.2" />
-      </geometry>
-    </collision>
-    <collision>
-      <origin xyz="0.01300000000000049 0.8170000000000014 -0.05125000000000081" rpy="3.14159265359 1.22464679915e-16 3.14159265359" />
-      <geometry>
-        <cylinder radius="0.05" length="0.0125" />
-      </geometry>
-    </collision>
-    <collision>
-      <origin xyz="-0.011999999999999594 0.7480000000000013 -0.051250000000000746" rpy="3.14159265359 1.22464679915e-16 3.14159265359" />
-      <geometry>
-        <cylinder radius="0.045" length="0.0125" />
-      </geometry>
-    </collision>
-    <collision>
-      <origin xyz="0.03600000000000049 0.7250000000000013 -0.051250000000000726" rpy="1.57079632679 1.08801856413e-14 -2.53072741539" />
-      <geometry>
-        <box size="0.08 0.0125 0.15" />
-      </geometry>
-    </collision>
-    <collision>
-      <origin xyz="0.04600000000000061 0.9000000000000016 -0.051250000000000885" rpy="1.57079632679 -1.54140589181e-13 2.96705972839" />
-      <geometry>
-        <box size="0.04 0.0125 0.15" />
-      </geometry>
-    </collision>
-    <collision>
-      <origin xyz="-0.0269999999999996 0.7900000000000014 -0.05125000000000078" rpy="1.57079632679 -9.51877465738e-14 2.91469985083" />
-      <geometry>
-        <box size="0.02 0.0125 0.03" />
-      </geometry>
-    </collision>
-    <collision>
-      <origin xyz="0.01300000000000049 0.8170000000000012 0.05124999999999934" rpy="3.14159265359 1.22464679915e-16 3.14159265359" />
-      <geometry>
-        <cylinder radius="0.05" length="0.0125" />
-      </geometry>
-    </collision>
-    <collision>
-      <origin xyz="-0.011999999999999594 0.7480000000000011 0.0512499999999994" rpy="3.14159265359 1.22464679915e-16 3.14159265359" />
-      <geometry>
-        <cylinder radius="0.045" length="0.0125" />
-      </geometry>
-    </collision>
-    <collision>
-      <origin xyz="0.03600000000000049 0.7250000000000011 0.05124999999999942" rpy="1.57079632679 1.08801856413e-14 -2.53072741539" />
-      <geometry>
-        <box size="0.08 0.0125 0.15" />
-      </geometry>
-    </collision>
-    <collision>
-      <origin xyz="0.04600000000000061 0.9000000000000014 0.05124999999999926" rpy="1.57079632679 -1.54140589181e-13 2.96705972839" />
-      <geometry>
-        <box size="0.04 0.0125 0.15" />
-      </geometry>
-    </collision>
-    <collision>
-      <origin xyz="-0.0269999999999996 0.7900000000000011 0.051249999999999366" rpy="1.57079632679 -9.51877465738e-14 2.91469985083" />
-      <geometry>
-        <box size="0.02 0.0125 0.03" />
-      </geometry>
-    </collision>
-    <collision>
-      <origin xyz="0.08000000000000103 1.4800000000000024 -0.060000000000001434" rpy="3.14159265359 1.22464679915e-16 3.14159265359" />
-      <geometry>
-        <cylinder radius="0.035" length="0.014" />
-      </geometry>
-    </collision>
-    <collision>
-      <origin xyz="0.09275648678445134 1.4111721564705255 -0.06000000000000137" rpy="1.57079632679 1.36016198304e-13 -2.95833308213" />
-      <geometry>
-        <box size="0.07 0.014 0.14" />
-      </geometry>
-    </collision>
-    <collision>
-      <origin xyz="0.07755703523082591 1.4100426421086656 -0.06000000000000137" rpy="1.57079632679 -3.49884704542e-12 3.10668606855" />
-      <geometry>
-        <box size="0.07 0.014 0.14" />
-      </geometry>
-    </collision>
-    <collision>
-      <origin xyz="0.09050000000000097 1.340000000000002 -0.06000000000000131" rpy="1.57079632679 6.59507171097e-13 -3.06305283725" />
-      <geometry>
-        <box size="0.0995 0.014 0.02" />
-      </geometry>
-    </collision>
-    <collision>
-      <origin xyz="0.08000000000000103 1.4800000000000024 -0.05000000000000142" rpy="3.14159265359 1.22464679915e-16 3.14159265359" />
-      <geometry>
-        <cylinder radius="0.03" length="0.004" />
-      </geometry>
-    </collision>
-    <collision>
-      <origin xyz="0.08000000000000103 1.4800000000000022 0.05999999999999875" rpy="3.14159265359 1.22464679915e-16 3.14159265359" />
-      <geometry>
-        <cylinder radius="0.035" length="0.014" />
-      </geometry>
-    </collision>
-    <collision>
-      <origin xyz="0.09275648678445134 1.4111721564705253 0.05999999999999881" rpy="1.57079632679 1.36016198304e-13 -2.95833308213" />
-      <geometry>
-        <box size="0.07 0.014 0.14" />
-      </geometry>
-    </collision>
-    <collision>
-      <origin xyz="0.07755703523082591 1.4100426421086654 0.05999999999999881" rpy="1.57079632679 -3.49884704542e-12 3.10668606855" />
-      <geometry>
-        <box size="0.07 0.014 0.14" />
-      </geometry>
-    </collision>
-    <collision>
-      <origin xyz="0.09050000000000097 1.340000000000002 0.059999999999998874" rpy="1.57079632679 6.59507171097e-13 -3.06305283725" />
-      <geometry>
-        <box size="0.0995 0.014 0.02" />
-      </geometry>
-    </collision>
-    <collision>
-      <origin xyz="0.08000000000000103 1.4800000000000022 0.04999999999999874" rpy="3.14159265359 1.22464679915e-16 3.14159265359" />
-      <geometry>
-        <cylinder radius="0.03" length="0.004" />
-      </geometry>
-    </collision>
   </link>
   <link name="MANIARM">
+    <visual>
+      <material name="maniarm_color"/>
+      <geometry>
+        <mesh filename="package://double_arm_tnk_description/meshes/mani_arm_v7_2.stl"/>
+      </geometry>
+    </visual>
+    <collision>
+      <geometry>
+        <mesh filename="package://double_arm_tnk_description/meshes/mani_arm_v7_2.stl"/>
+      </geometry>
+    </collision>
     <inertial>
       <mass value="28.673428" />
@@ -191,12 +117,19 @@
       <inertia ixx="0.19152986" ixy="0.11443044" ixz="0.0" iyy="0.79632756" iyz="0.0" izz="0.81910511" />
     </inertial>
-    <visual>
-      <origin xyz="0.0 0.0 0.0" rpy="7.8859849469e-16 9.95799250103e-17 -1.57079632679" />
-      <geometry>
-        <mesh filename="package://double_arm_tnk_description/meshes/DoubleArmV7-Upper-MANIARM-visual-0.dae" scale="1.0000000000000013 1.000000000000002 1.0000000000000016" />
-      </geometry>
-    </visual>
   </link>
   <link name="MANIELBOW">
+    <visual>
+      <origin rpy="${-M_PI/2} ${-M_PI/2} 0"/>
+      <material name="manielbow_color"/>
+      <geometry>
+        <mesh filename="package://double_arm_tnk_description/meshes/mani_elbow_v7_marge.stl"/>
+      </geometry>
+    </visual>
+    <collision>
+      <origin rpy="${-M_PI/2} ${-M_PI/2} 0"/>
+      <geometry>
+        <mesh filename="package://double_arm_tnk_description/meshes/mani_elbow_v7_marge.stl"/>
+      </geometry>
+    </collision>
     <inertial>
       <mass value="1e-06" />
@@ -206,4 +139,17 @@
   </link>
   <link name="YAWJOINT">
+    <visual>
+      <origin rpy="0 ${-M_PI/2} ${M_PI/2}"/>
+      <material name="yawjoint_color"/>
+      <geometry>
+        <mesh filename="package://double_arm_tnk_description/meshes/mani_plan2_roll_v7.stl"/>
+      </geometry>
+    </visual>
+    <collision>
+      <origin rpy="0 ${-M_PI/2} 0"/>
+      <geometry>
+        <mesh filename="package://double_arm_tnk_description/meshes/mani_plan2_roll_v7.stl"/>
+      </geometry>
+    </collision>
     <inertial>
       <mass value="1e-06" />
@@ -213,4 +159,17 @@
   </link>
   <link name="HANDBASE">
+    <visual>
+      <origin rpy="0 ${-M_PI/2} 0"/>
+      <material name="handbase_color"/>
+      <geometry>
+        <mesh filename="package://double_arm_tnk_description/meshes/handbase_marge_v7.stl"/>
+      </geometry>
+    </visual>
+    <collision>
+      <origin rpy="0 ${-M_PI/2} 0"/>
+      <geometry>
+        <mesh filename="package://double_arm_tnk_description/meshes/handbase_marge_v7.stl"/>
+      </geometry>
+    </collision>
     <inertial>
       <mass value="1e-06" />
@@ -220,4 +179,11 @@
   </link>
   <link name="PUSHROD">
+    <visual>
+      <origin rpy="0 ${-M_PI/2} 0"/>
+      <material name="pushrod_color"/>
+      <geometry>
+        <mesh filename="package://double_arm_tnk_description/meshes/hand_rod_v7.stl"/>
+      </geometry>
+    </visual>
     <inertial>
       <mass value="1e-06" />
@@ -227,4 +193,17 @@
   </link>
   <link name="HANDSLNK_I">
+    <visual>
+      <origin rpy="0 0 ${61.2291*M_PI/180}"/>
+      <material name="handslnk_i_color"/>
+      <geometry>
+        <mesh filename="package://double_arm_tnk_description/meshes/hand_slink_inner_v7.stl"/>
+      </geometry>
+    </visual>
+    <collision>
+      <origin rpy="0 0 ${61.2291*M_PI/180}"/>
+      <geometry>
+        <mesh filename="package://double_arm_tnk_description/meshes/hand_slink_inner_v7.stl"/>
+      </geometry>
+    </collision>
     <inertial>
       <mass value="0.408083" />
@@ -232,30 +211,19 @@
       <inertia ixx="0.000186599" ixy="0.0" ixz="0.0" iyy="0.000536909" iyz="0.0" izz="0.000414755" />
     </inertial>
-    <visual>
-      <origin xyz="0.0 0.0 0.0" rpy="-1.35515238445e-15 -1.57079632679 0.0" />
-      <geometry>
-        <mesh filename="package://double_arm_tnk_description/meshes/DoubleArmV7-Upper-HANDSLNK_I-visual-0.dae" scale="1.000000000000002 1.0000000000000016 1.0000000000000022" />
-      </geometry>
-    </visual>
-    <collision>
-      <origin xyz="-4.898587196589429e-18 -4.839211798541819e-17 0.040000000000000084" rpy="-1.35515238445e-15 -1.57079632679 0.0" />
-      <geometry>
-        <box size="0.08 0.028 0.028" />
-      </geometry>
-    </collision>
-    <collision>
-      <origin xyz="0.0 0.0 0.0" rpy="3.14159265359 -1.57079632679 0.0" />
-      <geometry>
-        <cylinder radius="0.014" length="0.028" />
-      </geometry>
-    </collision>
-    <collision>
-      <origin xyz="-9.797174393178858e-18 -9.678423597083638e-17 0.08000000000000017" rpy="3.14159265359 -1.57079632679 0.0" />
-      <geometry>
-        <cylinder radius="0.014" length="0.028" />
-      </geometry>
-    </collision>
   </link>
   <link name="HANDSLNK_O">
+    <visual>
+      <origin rpy="0 0 ${-61.2291*M_PI/180}"/>
+      <material name="handslnk_o_color"/>
+      <geometry>
+        <mesh filename="package://double_arm_tnk_description/meshes/hand_slink_outer_v7.stl"/>
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
Commit message: Update to add transform info

File: double_arm_tnk_description/urdf/MANI_ARM.urdf.xacro (robot description, xacro)
@@ -360,4 +360,5 @@
     <limit lower="-11.9991386075" upper="11.9991386075" effort="12000.0" velocity="573.0" />
   </joint>
+  <xacro:joint_trans_v0 name="UFRAME"/>
   <joint name="MNP_SWING" type="revolute">
     <origin xyz="0.5595 -0.13 0.11800000000000005" rpy="0.0 -0.0 0.0" />
@@ -367,4 +368,5 @@
     <limit lower="-1.0471975512" upper="1.0471975512" effort="12000.0" velocity="1146.0" />
   </joint>
+  <xacro:joint_trans_v0 name="MNP_SWING"/>
   <joint name="MANIBOOM" type="revolute">
     <origin xyz="0.07000000000000028 1.942890293094024e-16 0.1400000000000003" rpy="-1.57079632679 1.57079632679 0.0" />
@@ -374,4 +376,5 @@
     <limit lower="0.0" upper="2.00712863979" effort="15000.0" velocity="573.0" />
   </joint>
+  <xacro:joint_trans_v0 name="MANIBOOM"/>
   <joint name="MANIARM" type="revolute">
     <origin xyz="-1.4799999999999995 0.0800000000000003 -4.718447854656915e-16" rpy="0.0 -0.0 3.14159265359" />
@@ -381,4 +384,5 @@
     <limit lower="-1.91986217719" upper="0.0" effort="12000.0" velocity="573.0" />
   </joint>
+  <xacro:joint_trans_v0 name="MANIARM"/>
   <joint name="MANIELBOW" type="revolute">
     <origin xyz="-0.5499999999999989 0.27000000000000035 1.942890293094024e-16" rpy="1.57079632679 1.16573417586e-15 1.57079632679" />
@@ -388,4 +392,5 @@
     <limit lower="-1.57079632679" upper="0.349065850399" effort="10000.0" velocity="573.0" />
   </joint>
+  <xacro:joint_trans_v0 name="MANIELBOW"/>
   <joint name="YAWJOINT" type="revolute">
     <origin xyz="-4.440892098500626e-16 5.273559366969494e-16 -0.2300000000000002" rpy="0.0 -0.0 0.0" />
@@ -395,4 +400,5 @@
     <limit lower="-0.881042206407" upper="0.881042206407" effort="10000.0" velocity="573.0" />
   </joint>
+  <xacro:joint_trans_v0 name="YAWJOINT"/>
   <joint name="HANDBASE" type="revolute">
     <origin xyz="-4.440892098500626e-16 -2.7755575615628914e-17 -0.40529999999999977" rpy="0.0 -0.0 0.0" />
@@ -402,4 +408,5 @@
     <limit lower="-4.71238898038" upper="4.71238898038" effort="8000.0" velocity="573.0" />
   </joint>
+  <xacro:joint_trans_v0 name="HANDBASE"/>
   <joint name="PUSHROD" type="prismatic">
     <origin xyz="-1.1102230246251565e-16 -2.7755575615628914e-17 -0.0917" rpy="0.0 -0.0 0.0" />
@@ -409,4 +416,5 @@
     <limit lower="-0.000884881930761" upper="0.0" effort="8000.0" velocity="573.0" />
   </joint>
+  <xacro:joint_trans_v0 name="PUSHROD"/>
   <joint name="HANDSLNK_I" type="revolute">
     <origin xyz="1.1102230246251565e-16 3.885780586188048e-16 1.1102230246251565e-16" rpy="-1.57079632679 0.502146933762 3.14159265359" />

File: double_arm_tnk_description/urdf/TOHOKU_ARM.urdf.xacro (robot description, xacro)
@@ -1,5 +1,6 @@
 <?xml version="1.0"?>
-<robot  xmlns:xacro="http://ros.org/wiki/xacro">
-  <!-- == Material == -->
+<robot xmlns:xacro="http://ros.org/wiki/xacro">
+  <xacro:include filename="$(find double_arm_tnk_description)/urdf/common.xacro"/>
+    <!-- == Material == -->
   <material name="mframe_color">
     <color rgba="0.2 0.2 0.2 1"/>
@@ -188,4 +189,5 @@
     <limit lower="-11.9991386075" upper="11.9991386075" effort="12000.0" velocity="180.0" />
   </joint>
+  <xacro:joint_trans_v0 name="MFRAME"/>
   <joint name="BLOCK" type="revolute">
     <origin xyz="0.845 -0.11 0.192" rpy="0.0 -0.0 0.0" />
@@ -195,4 +197,5 @@
     <limit lower="-0.837758040957" upper="1.21300383014" effort="12000.0" velocity="1146.0" />
   </joint>
+  <xacro:joint_trans_v0 name="BLOCK"/>
   <joint name="BOOM" type="revolute">
     <origin xyz="0.0700000000000004 1.5265566588595902e-16 0.20000000000000012" rpy="1.57079632679 8.65956056235e-17 3.14159265359" />
@@ -202,4 +205,5 @@
     <limit lower="-1.31074226825" upper="0.928515162061" effort="15000.0" velocity="1146.0" />
   </joint>
+  <xacro:joint_trans_v0 name="BOOM"/>
   <joint name="ARM" type="revolute">
     <origin xyz="-1.7599999999999993 5.551115123125783e-16 -9.71445146547012e-17" rpy="0.0 -0.0 0.0" />
@@ -209,4 +213,5 @@
     <limit lower="0.535816080362" upper="2.65464579228" effort="12000.0" velocity="1146.0" />
   </joint>
+  <xacro:joint_trans_v0 name="ARM"/>
   <joint name="TOHKU_PITCH" type="revolute">
     <origin xyz="-0.9649999999999999 1.6653345369377348e-16 -5.551115123125783e-17" rpy="1.57079632679 -1.11022302463e-16 1.57079632679" />
@@ -216,4 +221,5 @@
     <limit lower="-0.588175957922" upper="1.57079632679" effort="10000.0" velocity="5730.0" />
   </joint>
+  <xacro:joint_trans_v0 name="TOHKU_ROLL"/>
   <joint name="TOHKU_ROLL" type="revolute">
     <origin xyz="9.992007221626409e-16 1.3183898417423734e-15 -0.22699999999999942" rpy="0.0 -0.0 0.0" />
@@ -223,4 +229,5 @@
     <limit lower="-3.14159265359" upper="3.14159265359" effort="10000.0" velocity="573.0" />
   </joint>
+  <xacro:joint_trans_v0 name="TOHKU_PITCH"/>
   <joint name="TOHKU_TIP_01" type="revolute">
     <origin xyz="9.992007221626409e-16 -7.077671781985373e-16 -0.3089999999999997" rpy="0.0 -0.0 0.0" />
@@ -230,4 +237,5 @@
     <limit lower="-0.349065850399" upper="0.0" effort="10000.0" velocity="573.0" />
   </joint>
+  <xacro:joint_trans_v0 name="TOHKU_TIP_01"/>
   <joint name="TOHKU_TIP_02" type="revolute">
     <origin xyz="9.992007221626409e-16 -7.077671781985373e-16 -0.3089999999999997" rpy="0.0 -0.0 3.14159265359" />
@@ -237,3 +245,4 @@
     <limit lower="-0.349065850399" upper="0.0" effort="10000.0" velocity="573.0" />
   </joint>
+  <xacro:joint_trans_v0 name="TOHKU_TIP_02"/>
 </robot>

File: double_arm_tnk_description/urdf/common.xacro (robot description, xacro)
@@ -1,5 +1,5 @@
 <?xml version="1.0"?>
 <robot xmlns:xacro="http://ros.org/wiki/xacro">
-  <property name="M_PI" value="3.14159274"/>
+  <xacro:property name="M_PI" value="3.14159274"/>
   <xacro:macro name="cylinder_inertial" params="mass radius length">
 	<mass value="${mass}"/>
@@ -14,3 +14,14 @@
 			 izz="${(mass*(height*height+width*width))/12}" />
   </xacro:macro>
+  <xacro:macro name="joint_trans_v0" params="name">
+	<transmission name="${name}_trans">
+      <type>transmission_interface/SimpleTransmission</type>
+      <joint name="${name}">
+		<hardwareInterface>PositionJointInterface</hardwareInterface>
+      </joint>
+	  <actuator name="${name}_motor">
+		<hardwareInterface>PositionJointInterface</hardwareInterface>
+      </actuator>
+	</transmission>
+  </xacro:macro>
 </robot>
