Commit message: Update delete each material colors

File: double_arm_tnk_description/urdf/common.xacro (robot description, xacro)
@@ -14,9 +14,3 @@
 			 izz="${(mass*(height*height+width*width))/12}" />
   </xacro:macro>
-  <material name="wheel_color">
-    <color rgba="0.3 0.3 0.3 1"/>
-  </material>
-  <material name="tframe_color">
-    <color rgba="0.3 0.3 0.3 0.8"/>
-  </material>
 </robot>

Commit message: Update add velocity transmission macro

File: double_arm_tnk_description/urdf/common.xacro (robot description, xacro)
@@ -25,3 +25,14 @@
 	</transmission>
   </xacro:macro>
+  <xacro:macro name="joint_velocity_trans_v0" params="name">
+	<transmission name="${name}_trans">
+      <type>transmission_interface/SimpleTransmission</type>
+      <joint name="${name}">
+		<hardwareInterface>VelocityJointInterface</hardwareInterface>
+      </joint>
+	  <actuator name="${name}_motor">
+		<hardwareInterface>VelocityJointInterface</hardwareInterface>
+      </actuator>
+	</transmission>
+  </xacro:macro>
 </robot>
