Commit message: Update delete unnecessary part

File: double_arm_tnk_description/urdf/BASE.urdf.xacro (robot description, xacro)
@@ -116,6 +116,4 @@
   <link name="WIRE_GUARD_L">
     <visual>
-      <!-- <origin xyz="0.02 0.61 -0.32" rpy="0.0 -0.0 0.0" /> -->
-      <!-- <origin xyz="0.26 0.6 -0.295" rpy="0.0 -0.0 0.0" /> -->
       <origin xyz="0.72 -0.01 0.0255" rpy="${M_PI/2} 0 0"/>
       <material name="tframe_color"/>

Commit message: Update material color

File: double_arm_tnk_description/urdf/BASE.urdf.xacro (robot description, xacro)
@@ -1,4 +1,14 @@
 <?xml version="1.0"?>
 <robot xmlns:xacro="http://ros.org/wiki/xacro">
+  <!-- == Material == -->
+  <material name="wheel_color">
+    <color rgba="0.3 0.3 0.3 1"/>
+  </material>
+  <material name="wheel_guard_color">
+    <color rgba="0.3 0.3 0.3 0.8"/>
+  </material>
+  <material name="tframe_color">
+    <color rgba="0.3 0.3 0.3 1"/>
+  </material>
   <!-- Link -->
   <link name="WHEEL_L0">
@@ -117,5 +127,5 @@
     <visual>
       <origin xyz="0.72 -0.01 0.0255" rpy="${M_PI/2} 0 0"/>
-      <material name="tframe_color"/>
+      <material name="wheel_guard_color"/>
       <geometry>
         <mesh filename="package://double_arm_tnk_description/meshes/tframe.stl"/>
@@ -137,5 +147,5 @@
     <visual>
       <origin xyz="0.72 0.01 0.0255" rpy="${M_PI/2} 0 0"/>
-      <material name="tframe_color"/>
+      <material name="wheel_guard_color"/>
       <geometry>
         <mesh filename="package://double_arm_tnk_description/meshes/tframe.stl"/>

Commit message: Update set wheel joints as fixed joints

File: double_arm_tnk_description/urdf/BASE.urdf.xacro (robot description, xacro)
@@ -185,49 +185,41 @@
   </link>
   <!-- Joint -->
-  <joint name="WHEEL_L0" type="continuous">
+  <joint name="WHEEL_L0" type="fixed">
     <origin xyz="0.74 0.6 -0.295" rpy="0.0 -0.0 0.0" />
-    <axis xyz="0 1 0" />
     <parent link="TFRAME" />
     <child link="WHEEL_L0" />
   </joint>
-  <joint name="WHEEL_L1" type="continuous">
+  <joint name="WHEEL_L1" type="fixed">
     <origin xyz="0.26 0.6 -0.295" rpy="0.0 -0.0 0.0" />
-    <axis xyz="0 1 0" />
     <parent link="TFRAME" />
     <child link="WHEEL_L1" />
   </joint>
-  <joint name="WHEEL_L2" type="continuous">
+  <joint name="WHEEL_L2" type="fixed">
     <origin xyz="-0.22 0.6 -0.295" rpy="0.0 -0.0 0.0" />
-    <axis xyz="0 1 0" />
     <parent link="TFRAME" />
     <child link="WHEEL_L2" />
   </joint>
-  <joint name="WHEEL_L3" type="continuous">
+  <joint name="WHEEL_L3" type="fixed">
     <origin xyz="-0.7 0.6 -0.295" rpy="0.0 -0.0 0.0" />
-    <axis xyz="0 1 0" />
     <parent link="TFRAME" />
     <child link="WHEEL_L3" />
   </joint>
-  <joint name="WHEEL_R0" type="continuous">
+  <joint name="WHEEL_R0" type="fixed">
     <origin xyz="0.74 -0.6 -0.295" rpy="0.0 -0.0 0.0" />
-    <axis xyz="0 1 0" />
     <parent link="TFRAME" />
     <child link="WHEEL_R0" />
   </joint>
-  <joint name="WHEEL_R1" type="continuous">
+  <joint name="WHEEL_R1" type="fixed">
     <origin xyz="0.26 -0.6 -0.295" rpy="0.0 -0.0 0.0" />
-    <axis xyz="0 1 0" />
     <parent link="TFRAME" />
     <child link="WHEEL_R1" />
   </joint>
-  <joint name="WHEEL_R2" type="continuous">
+  <joint name="WHEEL_R2" type="fixed">
     <origin xyz="-0.22 -0.6 -0.295" rpy="0.0 -0.0 0.0" />
-    <axis xyz="0 1 0" />
     <parent link="TFRAME" />
     <child link="WHEEL_R2" />
   </joint>
-  <joint name="WHEEL_R3" type="continuous">
+  <joint name="WHEEL_R3" type="fixed">
     <origin xyz="-0.7 -0.6 -0.295" rpy="0.0 -0.0 0.0" />
-    <axis xyz="0 1 0" />
     <parent link="TFRAME" />
     <child link="WHEEL_R3" />

Commit message: Update to add transmission for wheels

File: double_arm_tnk_description/urdf/BASE.urdf.xacro (robot description, xacro)
@@ -185,9 +185,11 @@
   </link>
   <!-- Joint -->
-  <joint name="WHEEL_L0" type="fixed">
+  <joint name="WHEEL_L0" type="continuous">
     <origin xyz="0.74 0.6 -0.295" rpy="0.0 -0.0 0.0" />
     <parent link="TFRAME" />
     <child link="WHEEL_L0" />
-  </joint>
+    <axis xyz="0 -1 0"/>
+  </joint>
+  <xacro:joint_velocity_trans_v0 name="WHEEL_L0"/>
   <joint name="WHEEL_L1" type="fixed">
     <origin xyz="0.26 0.6 -0.295" rpy="0.0 -0.0 0.0" />
@@ -205,9 +207,11 @@
     <child link="WHEEL_L3" />
   </joint>
-  <joint name="WHEEL_R0" type="fixed">
+  <joint name="WHEEL_R0" type="continuous">
     <origin xyz="0.74 -0.6 -0.295" rpy="0.0 -0.0 0.0" />
     <parent link="TFRAME" />
     <child link="WHEEL_R0" />
-  </joint>
+    <axis xyz="0 -1 0"/>
+  </joint>
+  <xacro:joint_velocity_trans_v0 name="WHEEL_R0"/>
   <joint name="WHEEL_R1" type="fixed">
     <origin xyz="0.26 -0.6 -0.295" rpy="0.0 -0.0 0.0" />
